File: hardware/patcom.kicad_pcb (KiCad board)
At the start: 2 copper layers, 80 x 86 mm, 26 parts, among them SW1 SW_Push_SPDT, SW2 SW_Push_SPDT, SW3 SW_Push_SPDT, SW4 SW_Push_SPDT, SW5 SW_Push_SPDT, SW6 SW_Push_SPDT, SW7 SW_Push_SPDT, SW8 SW_Push_SPDT, U1 R-78E3.3-1.0

Commit message: update pcb
Parts:
- removed the G*** at (120.7, 69.1)
Routing:
- net Net-(SW4-LED+): track 119.1 -> 32.9 mm, vias 0 -> 3
- net Net-(LED1-K): track 363.1 -> 314.2 mm, vias 0 -> 6
- net Net-(SW2-LED+): track 93.8 -> 50.6 mm, vias 0 -> 2
- net GND: track 107.2 -> 84.3 mm, vias 0 -> 2
- net Net-(SW8-LED+): track 91.5 -> 70.6 mm, vias 0 -> 2
- net Net-(SW7-LED+): track 71.3 -> 50.5 mm, vias 0 -> 2
- net Net-(A1-A4/SDA): track 72.1 -> 89.3 mm, vias 0 -> 4
- net Net-(A1-A5/SCL): track 56.3 -> 68.8 mm, vias 0 -> 4
- net Net-(A1-D13_SCK): track 87.9 -> 75.5 mm, vias 0 -> 2
- net Net-(SW6-B): track 54.8 -> 65.7 mm, vias 0 -> 2
- net Net-(SW8-B): track 56.3 -> 46.1 mm
- net Net-(SW5-B): track 71.8 -> 81.6 mm, vias 0 -> 2
- net Net-(SW3-LED+): track 26.6 -> 33.6 mm, vias 0 -> 3
- net Net-(SW1-B): track 40.9 -> 47.1 mm, vias 0 -> 2
- net Net-(A1-3.3V): track 91.5 -> 86.0 mm, vias 0 -> 4
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
Commit message: basic configurator
Parts:
- moved G*** 27.4 mm to (167.5, 136.5)
Routing:
- added copper zone on F.Cu, net +9V
- added copper zone on B.Cu, net GND
Other:
- board text added: "Packet Commander Version 2.1, Revision 3 Designed by Tyler Reckart, July 2025"
