File: hardware/patcom.kicad_sch (KiCad schematic)
At the start: 18 parts, among them SW1 SW_Push_SPDT, SW2 SW_Push_SPDT, SW3 SW_Push_SPDT, SW4 SW_Push_SPDT, SW5 SW_Push_SPDT, SW6 SW_Push_SPDT, SW7 SW_Push_SPDT, SW8 SW_Push_SPDT, U1 R-78E3.3-1.0

Commit message: basic configurator
Parts:
- removed D1: 1N4001, Diode_THT:D_DO-41_SOD81_P10.16mm_Horizontal, symbol Diode:1N4001
Connections:
- net +9V: now also C1.1, U1.1 (IN)
Changed lines of the file:
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@@
+	(wire
+		(pts
+			(xy 40.64 74.93) (xy 41.91 74.93)
+		)
+		(stroke
+			(width 0)
+			(type default)
+		)
+	)
 	(wire
 		(pts
@@
 	(wire
 		(pts
-			(xy 49.53 106.68) (xy 33.02 106.68)
+			(xy 49.53 106.68) (xy 40.64 106.68)
 		)
 		(stroke
@@
 		(pts
 			(xy 140.97 55.88) (xy 176.53 55.88)
-		)
-		(stroke
-			(width 0)
-			(type default)
-		)
-	)
-	(wire
-		(pts
-			(xy 40.64 74.93) (xy 41.91 74.93)
 		)
 		(stroke
@@
 	(symbol
 		(lib_id "power:GND")
-		(at 33.02 106.68 270)
+		(at 40.64 106.68 270)
 		(unit 1)
 		(exclude_from_sim no)
@@
 		(fields_autoplaced yes)
 		(property "Reference" "#PWR02"
-			(at 26.67 106.68 0)
+			(at 34.29 106.68 0)
 			(effects
 				(font
@@
 		)
 		(property "Value" "GND"
-			(at 29.21 106.6799 90)
+			(at 36.83 106.6799 90)
 			(effects
 				(font
@@
 		)
 		(property "Footprint" ""
-			(at 33.02 106.68 0)
+			(at 40.64 106.68 0)
 			(effects
 				(font
@@
 		)
 		(property "Datasheet" ""
-			(at 33.02 106.68 0)
+			(at 40.64 106.68 0)
 			(effects
 				(font
@@
 		)
 		(property "Description" "Power symbol creates a global label with name \"GND\" , ground"
-			(at 33.02 106.68 0)
+			(at 40.64 106.68 0)
 			(effects
 				(font
@@
 	(symbol
 		(lib_id "power:+9V")
-		(at 33.02 74.93 90)
+		(at 40.64 74.93 90)
 		(unit 1)
 		(exclude_from_sim no)
@@
 		(dnp no)
 		(property "Reference" "#PWR01"
-			(at 36.83 74.93 0)
+			(at 44.45 74.93 0)
 			(effects
 				(font
@@
 		)
 		(property "Value" "+9V"
-			(at 29.21 74.9299 90)
+			(at 36.83 74.9299 90)
 			(effects
 				(font
@@
 		)
 		(property "Footprint" ""
-			(at 33.02 74.93 0)
+			(at 40.64 74.93 0)
 			(effects
 				(font
@@
 		)
 		(property "Datasheet" ""
-			(at 33.02 74.93 0)
+			(at 40.64 74.93 0)
 			(effects
 				(font
@@
 		)
 		(property "Description" "Power symbol creates a global label with name \"+9V\""
-			(at 33.02 74.93 0)
+			(at 40.64 74.93 0)
 			(effects
 				(font
@@
 					(unit 1)
 				)
-			)
-		)
-	)
-	(symbol
-		(lib_id "Diode:1N4001")
-		(at 36.83 74.93 180)
-		(unit 1)
-		(exclude_from_sim no)
-		(in_bom yes)
-		(on_board yes)
-		(dnp no)
-		(fields_autoplaced yes)
-		(property "Reference" "D1"
-			(at 36.83 68.58 0)
-			(effects
-				(font
-					(size 1.27 1.27)
-				)
-			)
-		)
-		(property "Value" "1N4001"
-			(at 36.83 71.12 0)
-			(effects
-				(font
-					(size 1.27 1.27)
-				)
-			)
-		)
-		(property "Footprint" "Diode_THT:D_DO-41_SOD81_P10.16mm_Horizontal"
-			(at 36.83 74.93 0)
-			(effects
-				(font
-					(size 1.27 1.27)
-				)
-				(hide yes)
-			)
-		)
-		(property "Datasheet" "http://www.vishay.com/docs/88503/1n4001.pdf"
-			(at 36.83 74.93 0)
-			(effects
-				(font
-					(size 1.27 1.27)
-				)
-				(hide yes)
-			)
-		)
-		(property "Description" "50V 1A General Purpose Rectifier Diode, DO-41"
-			(at 36.83 74.93 0)
-			(effects
-				(font
-					(size 1.27 1.27)
-				)
-				(hide yes)
-			)
-		)
-		(property "Sim.Device" "D"
-			(at 36.83 74.93 0)
-			(effects
-				(font
-					(size 1.27 1.27)
-				)
-				(hide yes)
-			)
-		)
-		(property "Sim.Pins" "1=K 2=A"
-			(at 36.83 74.93 0)
-			(effects
-				(font
-					(size 1.27 1.27)
-				)
-				(hide yes)
-			)
-		)
-		(pin "2"
-		)
-		(pin "1"
-		)
-		(instances
-			(project "patcom"
-				(path "/35a22188-4fea-4692-971d-1c7b6cef4946"
-					(reference "D1")
-					(unit 1)
-				)
